File: nova75.kicad_sch (KiCad schematic)
At the start: 225 parts, among them J1 TYPE-C-31-M-12, J2 Conn_01x02, K1 KEYSW, K10 KEYSW, K11 KEYSW, K12 KEYSW, K13 KEYSW, K14 KEYSW, K15 KEYSW, K16 KEYSW, K17 KEYSW, K18 KEYSW, K19 KEYSW, K2 KEYSW, K20 KEYSW, K21 KEYSW, K22 KEYSW, K23 KEYSW, K24 KEYSW, K25 KEYSW, K26 KEYSW, K27 KEYSW, K28 KEYSW, K29 KEYSW, K3 KEYSW, K30 KEYSW, K31 KEYSW, K32 KEYSW, K33 KEYSW, K34 KEYSW, K35 KEYSW, K36 KEYSW, K37 KEYSW, K38 KEYSW, K39 KEYSW, K4 KEYSW, K40 KEYSW, K41 KEYSW, K42 KEYSW, K43 KEYSW, K44 KEYSW, K45 KEYSW, K46 KEYSW, K47 KEYSW, K48 KEYSW, K49 KEYSW, K5 KEYSW, K50 KEYSW, K51 KEYSW, K52 KEYSW, K53 KEYSW, K54 KEYSW, K55 KEYSW, K56 KEYSW, K57 KEYSW, K58 KEYSW, K59 KEYSW, K6 KEYSW, K60 KEYSW, K61 KEYSW, K62 KEYSW, K63 KEYSW, K64 KEYSW, K65 KEYSW, K66 KEYSW, K67 KEYSW, K68 KEYSW, K69 KEYSW, K7 KEYSW, K70 KEYSW, K71 KEYSW, K72 KEYSW, K73 KEYSW, K74 KEYSW, K75 KEYSW, K76 KEYSW, K77 KEYSW, K8 KEYSW, K9 KEYSW, SW1 SW_Push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

Commit message: Update PCB
Connections:
- net GND: now also FB1.1
- net GNDREF: now also FB1.2, J1.S1 (SHIELD); no longer FB1.1
Other:
- moved on the sheet: FB1
Changed lines of the file:
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@@
   (junction (at -203.2 91.44) (diameter 0) (color 0 0 0 0)
   )
+  (junction (at 26.67 73.66) (diameter 0) (color 0 0 0 0)
+  )
   (junction (at -96.52 81.28) (diameter 0) (color 0 0 0 0)
   )
@@
   (junction (at -299.72 81.28) (diameter 0) (color 0 0 0 0)
   )
+  (junction (at 34.29 73.66) (diameter 0) (color 0 0 0 0)
+  )
   (junction (at -116.84 81.28) (diameter 0) (color 0 0 0 0)
   )
@@
   (no_connect (at 177.8 99.695))
   (no_connect (at 177.8 97.155))
+  (wire (pts (xy 34.29 73.66) (xy 34.29 72.39))
+    (stroke (width 0) (type default) (color 0 0 0 0))
+  )
   (wire (pts (xy -101.6 71.12) (xy -101.6 52.07))
     (stroke (width 0) (type default) (color 0 0 0 0))
@@
     (stroke (width 0) (type default) (color 0 0 0 0))
   )
+  (wire (pts (xy 26.67 73.66) (xy 26.67 77.47))
+    (stroke (width 0) (type default) (color 0 0 0 0))
+  )
   (wire (pts (xy -203.2 52.07) (xy -203.2 71.12))
     (stroke (width 0) (type default) (color 0 0 0 0))
@@
     (stroke (width 0) (type default) (color 0 0 0 0))
   )
-  (wire (pts (xy 40.005 72.39) (xy 40.005 76.835))
+  (wire (pts (xy 40.005 73.66) (xy 40.005 77.47))
     (stroke (width 0) (type default) (color 0 0 0 0))
   )
@@
     (stroke (width 0) (type default) (color 0 0 0 0))
   )
+  (wire (pts (xy 33.02 73.66) (xy 34.29 73.66))
+    (stroke (width 0) (type default) (color 0 0 0 0))
+  )
   (wire (pts (xy 215.265 46.99) (xy 219.075 46.99))
     (stroke (width 0) (type default) (color 0 0 0 0))
@@
     (stroke (width 0) (type default) (color 0 0 0 0))
   )
-  (wire (pts (xy 32.385 76.835) (xy 32.385 73.66))
-    (stroke (width 0) (type default) (color 0 0 0 0))
-  )
   (wire (pts (xy 92.71 93.345) (xy 92.71 94.615))
     (stroke (width 0) (type default) (color 0 0 0 0))
@@
     (stroke (width 0) (type default) (color 0 0 0 0))
   )
-  (wire (pts (xy 26.67 73.66) (xy 27.305 73.66))
+  (wire (pts (xy 26.67 73.66) (xy 27.94 73.66))
     (stroke (width 0) (type default) (color 0 0 0 0))
   )
@@
     (stroke (width 0) (type default) (color 0 0 0 0))
   )
-  (wire (pts (xy 34.29 72.39) (xy 40.005 72.39))
+  (wire (pts (xy 34.29 73.66) (xy 40.005 73.66))
     (stroke (width 0) (type default) (color 0 0 0 0))
   )
@@
     (pin "2")
   )
-  (symbol (lib_id "Device:FerriteBead_Small") (at 29.845 73.66 270) (unit 1)
+  (symbol (lib_id "Device:FerriteBead_Small") (at 30.48 73.66 270) (unit 1)
     (in_bom yes) (on_board yes)
-    (property "Reference" "FB1" (id 0) (at 24.765 76.2 90)
+    (property "Reference" "FB1" (id 0) (at 29.21 76.835 90)
       (effects (font (size 1.27 1.27)) (justify left))
     )
-    (property "Value" "FerriteBead_Small" (id 1) (at 28.6132 76.2 0)
+    (property "Value" "FerriteBead_Small" (id 1) (at 29.2482 76.2 0)
       (effects (font (size 1.27 1.27)) (justify left) hide)
     )
-    (property "Footprint" "Inductor_SMD:L_0603_1608Metric" (id 2) (at 29.845 71.882 90)
+    (property "Footprint" "Inductor_SMD:L_0603_1608Metric" (id 2) (at 30.48 71.882 90)
       (effects (font (size 1.27 1.27)) hide)
     )
-    (property "Datasheet" "~" (id 3) (at 29.845 73.66 0)
+    (property "Datasheet" "~" (id 3) (at 30.48 73.66 0)
       (effects (font (size 1.27 1.27)) hide)
     )
-    (property "LCSC" "C98288" (id 4) (at 29.845 73.66 0)
+    (property "LCSC" "C98288" (id 4) (at 30.48 73.66 0)
       (effects (font (size 1.27 1.27)) hide)
     )
@@
     (pin "2")
   )
-  (symbol (lib_id "power:GNDREF") (at 32.385 76.835 0) (unit 1)
-    (in_bom yes) (on_board yes) (fields_autoplaced)
-    (property "Reference" "#PWR0101" (id 0) (at 32.385 83.185 0)
-      (effects (font (size 1.27 1.27)) hide)
-    )
-    (property "Value" "" (id 1) (at 32.385 81.915 0))
-    (property "Footprint" "" (id 2) (at 32.385 76.835 0)
-      (effects (font (size 1.27 1.27)) hide)
-    )
-    (property "Datasheet" "" (id 3) (at 32.385 76.835 0)
-      (effects (font (size 1.27 1.27)) hide)
-    )
-    (pin "1")
-  )
   (symbol (lib_id "projectlocal:Key_switch") (at -27.94 34.29 0) (unit 1)
     (in_bom yes) (on_board yes)
@@
   (symbol (lib_id "power:GNDREF") (at 215.265 58.42 0) (unit 1)
     (in_bom yes) (on_board yes) (fields_autoplaced)
-    (property "Reference" "#PWR?" (id 0) (at 215.265 64.77 0)
+    (property "Reference" "#PWR0103" (id 0) (at 215.265 64.77 0)
       (effects (font (size 1.27 1.27)) hide)
     )
@@
     (pin "2")
   )
-  (symbol (lib_id "power:GND") (at 40.005 76.835 0) (unit 1)
+  (symbol (lib_id "power:GND") (at 40.005 77.47 0) (unit 1)
     (in_bom yes) (on_board yes)
-    (property "Reference" "#PWR0102" (id 0) (at 40.005 83.185 0)
+    (property "Reference" "#PWR0102" (id 0) (at 40.005 83.82 0)
       (effects (font (size 1.27 1.27)) hide)
     )
-    (property "Value" "GND" (id 1) (at 40.005 80.645 0))
-    (property "Footprint" "" (id 2) (at 40.005 76.835 0)
+    (property "Value" "GND" (id 1) (at 40.005 81.28 0))
+    (property "Footprint" "" (id 2) (at 40.005 77.47 0)
       (effects (font (size 1.27 1.27)) hide)
     )
-    (property "Datasheet" "" (id 3) (at 40.005 76.835 0)
+    (property "Datasheet" "" (id 3) (at 40.005 77.47 0)
       (effects (font (size 1.27 1.27)) hide)
     )
@@
     (pin "2")
   )
+  (symbol (lib_id "power:GNDREF") (at 26.67 77.47 0) (unit 1)
+    (in_bom yes) (on_board yes)
+    (property "Reference" "#PWR0101" (id 0) (at 26.67 83.82 0)
+      (effects (font (size 1.27 1.27)) hide)
+    )
+    (property "Value" "GNDREF" (id 1) (at 26.67 81.28 0))
+    (property "Footprint" "" (id 2) (at 26.67 77.47 0)
+      (effects (font (size 1.27 1.27)) hide)
+    )
+    (property "Datasheet" "" (id 3) (at 26.67 77.47 0)
+      (effects (font (size 1.27 1.27)) hide)
+    )
+    (pin "1")
+  )
   (symbol (lib_id "projectlocal:Key_switch") (at -231.14 34.29 0) (unit 1)
     (in_bom yes) (on_board yes)
@@
       (reference "#PWR033") (unit 1) (value "GND") (footprint "")
     )
-    (path "/33de51e4-f43b-45b1-833b-e21d84d90255"
+    (path "/f65cdcd8-9c23-4f2c-b70c-3aa4106609dd"
       (reference "#PWR0101") (unit 1) (value "GNDREF") (footprint "")
     )
@@
     )
     (path "/786e2b53-a5d6-4881-a383-08fef40e85b0"
-      (reference "#PWR?") (unit 1) (value "GNDREF") (footprint "")
+      (reference "#PWR0103") (unit 1) (value "GNDREF") (footprint "")
     )
     (path "/0426741d-a4b1-4e5b-8360-c593e2aab144"
